File: bosch-kf163-pll.kicad_pcb (KiCad board)
At the start: 4 copper layers, 46 x 72 mm, 89 parts, among them J101 TGA, J201 S353/CDP18U42P, Q101 DTC143ZE, Q102 DTC143ZE, Q103 DTC143ZE, Q104 DTC143ZE, Q201 DTC143ZE, Q202 DTC143ZE, Q203 DTC143ZE, Q204 DTC143ZE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

Commit message: schematic/pcb update
Parts:
- removed Q214: DTC143ZE, Package_TO_SOT_SMD:SOT-523
- added C302: 10n, Capacitor_SMD:C_0603_1608Metric, B.Cu at (122.1, 104.0)
- added C303: 39n, Capacitor_SMD:C_0603_1608Metric, B.Cu at (122.1, 108.6)
- added C304: 1n, Capacitor_SMD:C_0603_1608Metric, B.Cu at (122.1, 111.6)
- added C306: 10n, Capacitor_SMD:C_0603_1608Metric, B.Cu at (112.6, 103.1)
- added C307: 39n, Capacitor_SMD:C_0603_1608Metric, B.Cu at (112.6, 107.7)
- added C308: 1n, Capacitor_SMD:C_0603_1608Metric, B.Cu at (112.6, 110.7)
- added J102: PROG, Connector_PinHeader_2.54mm:PinHeader_1x04_P2.54mm_Horizontal, F.Cu at (93.3, 83.3)
- added R115: 0, Resistor_SMD:R_0603_1608Metric, B.Cu at (91.2, 102.9)
- added R116: 0, Resistor_SMD:R_0603_1608Metric, B.Cu at (91.2, 100.3)
- added R117: 0, Resistor_SMD:R_0603_1608Metric, B.Cu at (91.2, 97.8)
- added R301: 5.1k, Resistor_SMD:R_0603_1608Metric, B.Cu at (122.1, 105.5)
- added R302: 4.7k, Resistor_SMD:R_0603_1608Metric, B.Cu at (122.1, 107.1)
- added R303: 4.7k, Resistor_SMD:R_0603_1608Metric, B.Cu at (122.1, 110.1)
- added R304: 10k, Resistor_SMD:R_0603_1608Metric, B.Cu at (119.3, 102.5)
- added R305: 5.1k, Resistor_SMD:R_0603_1608Metric, B.Cu at (112.6, 104.6)
- added R306: 4.7k, Resistor_SMD:R_0603_1608Metric, B.Cu at (112.6, 106.2)
- added R307: 4.7k, Resistor_SMD:R_0603_1608Metric, B.Cu at (112.6, 109.2)
- J101: moved to B.Cu
- U101, U202: footprint Package_SO:SO-16_3.9x9.9mm_P1.27mm -> Package_SO:SOIC-16_3.9x9.9mm_P1.27mm
- moved R113 40.9 mm to (131.2, 129.7)
- moved Q103 24.2 mm to (107.2, 118.5), turned to 90 degrees
- moved U302 13.3 mm to (108.3, 106.2), turned to -90 degrees
- moved Q104 12.4 mm to (100.2, 134.5), turned to 180 degrees
- moved C104 11.0 mm to (102.0, 93.6)
- moved C301 7.94 mm to (116.6, 111.6), turned to 0 degrees
- moved C105 7.32 mm to (102.0, 95.9)
- moved R112 6.35 mm to (91.2, 105.4)
- moved C305 4.65 mm to (107.1, 110.7), turned to 0 degrees
- moved U301 4.16 mm to (117.8, 107.1), turned to -90 degrees
- moved J101 2.54 mm to (94.6, 95.2), turned to 180 degrees
- moved Q102 2.41 mm to (102.6, 134.5)
- moved D209 2.29 mm to (96.6, 83.2)
- moved D201 1.71 mm to (95.4, 79.6), turned to 0 degrees
- moved R216 1.02 mm to (124.2, 65.7)
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Connections:
- J101 pad 1: /SQUELCH -> MIC
- J101 pad 10: +8V -> TX_FLAT
- J101 pad 11: Net-(J101-Pad11) -> /HUP
- J101 pad 12: /HUP -> TX_FLAT
- J101 pad 13: Net-(J101-Pad13) -> St2
- J101 pad 14: St2 -> RX_FLAT
- J101 pad 15: Net-(J101-Pad13) -> /D
- J101 pad 16: /D -> RX_FLAT
- J101 pad 17: +8V -> /C
- J101 pad 18: /C -> +8V
- J101 pad 19: Net-(D101-Pad1) -> /B
- J101 pad 2: M -> /SQUELCH
- J101 pad 20: /B -> Net-(D101-Pad1)
- J101 pad 21: GND -> /A
- J101 pad 22: /A -> GND
- J101 pad 23: Net-(J101-Pad23) -> St1
- J101 pad 24: St1 -> TX_NF
- J101 pad 25: Net-(J101-Pad23) -> /LED_GN
- J101 pad 26: /LED_GN -> TX_NF
- J101 pad 27: VDC -> /DEL
- J101 pad 28: /DEL -> VDC
- J101 pad 29: RXNF -> /CALL2
- J101 pad 3: SQL_SENSE -> Net-(J101-Pad3)
- J101 pad 30: /CALL2 -> RXNF
- J101 pad 31: Net-(J101-Pad31) -> /CALL1
- J101 pad 32: /CALL1 -> Net-(J101-Pad32)
- J101 pad 4: unconnected-(J101-Pad4) -> SQL_SENSE
- J101 pad 5: unconnected-(J101-Pad5) -> Net-(J101-Pad5)
- J101 pad 7: ONOFF -> Net-(J101-Pad7)
- J101 pad 8: Net-(J101-Pad8) -> ONOFF
- J101 pad 9: Net-(J101-Pad11) -> +8V
- Q102 pad 3: Net-(J101-Pad31) -> Net-(J101-Pad32)
- R113 pad 1: Net-(J101-Pad8) -> Net-(R113-Pad1)
- R113 pad 2: unconnected-(R113-Pad2) -> TXD
- U103 pad 35: TXD -> Net-(R113-Pad1)
- U202 pad 14: unconnected-(U202-Pad14) -> GND
Routing:
- net BOOT: track 0.00 -> 89.5 mm, vias 0 -> 2
- net RXD: track 0.00 -> 80.5 mm, vias 0 -> 1
- net TXD: track 0.00 -> 78.7 mm, vias 0 -> 1
- net Net-(D205-Pad1): track 30.9 -> 100.2 mm, vias 0 -> 2
- net Net-(D212-Pad1): track 33.6 -> 99.4 mm, vias 0 -> 2
- net LATCH: track 69.0 -> 127.6 mm, vias 2 -> 4
- net CLK: track 69.7 -> 123.5 mm, vias 2 -> 4
- net Net-(D204-Pad1): track 29.6 -> 72.2 mm, vias 0 -> 1
- net Net-(D211-Pad1): track 25.3 -> 64.1 mm, vias 0 -> 1
- net MOSI: track 0.00 -> 38.4 mm
- net Net-(D203-Pad1): track 25.0 -> 63.2 mm, vias 0 -> 1
- net Net-(D202-Pad1): track 24.3 -> 61.9 mm, vias 0 -> 1
- net Net-(D210-Pad1): track 24.9 -> 62.4 mm, vias 0 -> 1
- net Net-(D103-Pad1): track 0.00 -> 35.4 mm, vias 0 -> 2
- net +3V3: track 124.5 -> 158.3 mm, vias 12 -> 18
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Other:
- board text added: "D"
- board text added: "U"
- board text added: "X"

Commit message: schematic/pcb update
Parts:
- added C309: 10u, Capacitor_SMD:C_0603_1608Metric, B.Cu at (111.4, 103.2)
- added C310: 10u, Capacitor_SMD:C_0603_1608Metric, B.Cu at (100.8, 109.2)
- added C311: 10u, Capacitor_SMD:C_0603_1608Metric, B.Cu at (100.8, 107.7)
- added C312: 10u, Capacitor_SMD:C_0603_1608Metric, B.Cu at (100.8, 112.3)
- added C313: 10u, Capacitor_SMD:C_0603_1608Metric, B.Cu at (100.8, 110.7)
- added C314: 10u, Capacitor_SMD:C_0603_1608Metric, B.Cu at (125.1, 111.8)
- added C315: 10u, Capacitor_SMD:C_0603_1608Metric, B.Cu at (122.8, 103.4)
- added Q214: DTC143ZE, Package_TO_SOT_SMD:SOT-523, B.Cu at (128.9, 68.6)
- added R308: 4.7k, Resistor_SMD:R_0603_1608Metric, B.Cu at (109.9, 103.2)
- added R309: 4.7k, Resistor_SMD:R_0603_1608Metric, B.Cu at (108.3, 103.2)
- added R310: 4.7k, Resistor_SMD:R_0603_1608Metric, B.Cu at (126.6, 108.7)
- added R311: 4.7k, Resistor_SMD:R_0603_1608Metric, B.Cu at (125.1, 108.7)
- added R312: 4.7k, Resistor_SMD:R_0603_1608Metric, B.Cu at (125.9, 103.4)
- added R313: 4.7k, Resistor_SMD:R_0603_1608Metric, B.Cu at (126.6, 111.8)
- added R314: 4.7k, Resistor_SMD:R_0603_1608Metric, B.Cu at (125.1, 105.7)
- added R315: 4.7k, Resistor_SMD:R_0603_1608Metric, B.Cu at (126.6, 105.7)
- added RV301: 50k, Potentiometer_SMD:Potentiometer_Bourns_TC33X_Vertical, F.Cu at (109.2, 106.6)
- added RV302: 50k, Potentiometer_SMD:Potentiometer_Bourns_TC33X_Vertical, F.Cu at (124.3, 106.8)
- C104, C105: value 100n -> 10u
- J201: footprint Package_DIP:DIP-28_W15.24mm_LongPads -> Package_DIP:DIP-28_W15.24mm_Socket_LongPads; moved to B.Cu
- R304: value 10k -> 4.7k
- moved C304 15.3 mm to (106.8, 111.8), turned to -90 degrees
- moved J201 15.2 mm to (132.1, 66.0), turned to 180 degrees
- moved C306 14.0 mm to (123.6, 111.8), turned to 90 degrees
- moved R303 13.9 mm to (108.3, 111.8), turned to 90 degrees
- moved C305 13.6 mm to (118.9, 103.9)
- moved C303 12.7 mm to (109.9, 111.8), turned to 90 degrees
- moved U302 12.3 mm to (120.5, 107.4), turned to 180 degrees
- moved R305 11.8 mm to (122.0, 111.8), turned to -90 degrees
- moved R302 11.7 mm to (111.4, 111.8), turned to -90 degrees
- moved C301 11.2 mm to (106.8, 106.3), turned to -90 degrees
- moved R301 11.1 mm to (112.9, 111.8), turned to -90 degrees
- moved C302 10.9 mm to (114.4, 111.8), turned to 90 degrees
- moved R306 9.71 mm to (120.5, 111.8), turned to -90 degrees
- moved C307 7.59 mm to (119.0, 111.8), turned to 90 degrees
- moved R304 7.07 mm to (116.0, 108.7), turned to 90 degrees
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Connections:
- C307 pad 2: Net-(C307-Pad2) -> ADC1
- J101 pad 30: RXNF -> RX_NF
- R116 pad 2: RXD -> TXD
- R117 pad 2: TXD -> RXD
- U302 pad 2: unconnected-(U302-Pad2) -> Net-(R314-Pad1)
- U302 pad 3: unconnected-(U302-Pad3) -> Net-(C312-Pad2)
- U302 pad 6: Net-(C307-Pad2) -> ADC1
- U302 pad 7: Net-(C307-Pad2) -> ADC1
Routing:
- net +3V3: track 158.3 -> 268.4 mm, vias 18 -> 35
- net RXNF: track 33.7 -> 0.00 mm, vias 1 -> 0
- net SQL_SENSE: track 11.2 -> 44.8 mm, vias 0 -> 2
- net RX_NF: track 0.00 -> 32.1 mm, vias 0 -> 1
- net Net-(C312-Pad2): track 0.00 -> 27.2 mm, vias 0 -> 2
- net +8V: track 27.6 -> 52.0 mm, vias 0 -> 2
- net GND: track 73.1 -> 90.7 mm, vias 50 -> 113
- net Net-(C310-Pad1): track 0.00 -> 15.4 mm, vias 0 -> 1
- net ADC1: track 13.0 -> 24.3 mm, vias 1 -> 2
- net Net-(R305-Pad1): track 6.92 -> 16.1 mm, vias 0 -> 1
- net MOSI: track 38.4 -> 30.6 mm
- net Net-(R314-Pad1): track 0.00 -> 6.56 mm, vias 0 -> 1
- net MISO_PLL: track 71.0 -> 77.4 mm
- net Net-(C307-Pad2): track 5.70 -> 0.00 mm
- net DAC1: track 13.5 -> 18.7 mm, vias 1 -> 2
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- added copper zone on B.Cu, net +3V3
- added copper zone on In1.Cu, net +3V3
