File: filter.kicad_sch (KiCad schematic)
At the start: 34 parts, among them U301 RS8752XK, U302 RS8752XK

Commit message: sheet comments, schematic variants, removed txd resistor
Parts:
- C301, C302, C303, C304, C305, C306, C307, C308, C309, C310, C311, C312, C313, C314, C315, R301, R302, R303, R304, R305, R306, R307, R310, R311, R312, R313, RV301, RV302, U301, U302: variant (none) -> Audio
- R308, R309, R314, R315: DNP (none) -> DNP; variant (none) -> Audio
Changed lines of the file:
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@@
+      (effects (font (size 1.27 1.27)) hide)
+    )
+    (property "variant" "Audio" (id 5) (at 158.75 109.22 0)
       (effects (font (size 1.27 1.27)) hide)
     )
@@
       (effects (font (size 1.27 1.27)) hide)
     )
+    (property "variant" "Audio" (id 5) (at 85.09 125.73 0)
+      (effects (font (size 1.27 1.27)) hide)
+    )
     (pin "1")
     (pin "2")
@@
       (effects (font (size 1.27 1.27)) hide)
     )
+    (property "variant" "Audio" (id 5) (at 135.89 119.38 0)
+      (effects (font (size 1.27 1.27)) hide)
+    )
     (pin "1")
     (pin "2")
@@
     )
     (property "LCSC" "C105428" (id 4) (at 85.09 135.89 0)
+      (effects (font (size 1.27 1.27)) hide)
+    )
+    (property "variant" "Audio" (id 5) (at 85.09 135.89 0)
       (effects (font (size 1.27 1.27)) hide)
     )
@@
       (effects (font (size 1.27 1.27)) hide)
     )
+    (property "variant" "Audio" (id 5) (at 105.41 48.26 0)
+      (effects (font (size 1.27 1.27)) hide)
+    )
     (pin "1")
     (pin "2")
@@
     )
     (property "LCSC" "C2922482" (id 4) (at 135.89 143.51 0)
+      (effects (font (size 1.27 1.27)) hide)
+    )
+    (property "variant" "Audio" (id 5) (at 135.89 143.51 0)
       (effects (font (size 1.27 1.27)) hide)
     )
@@
       (effects (font (size 1.27 1.27)) hide)
     )
+    (property "variant" "Audio" (id 5) (at 177.8 55.88 0)
+      (effects (font (size 1.27 1.27)) hide)
+    )
     (pin "1")
     (pin "2")
@@
       (effects (font (size 1.27 1.27)) hide)
     )
+    (property "variant" "Audio" (id 5) (at 66.04 43.18 0)
+      (effects (font (size 1.27 1.27)) hide)
+    )
     (pin "1")
     (pin "2")
@@
       (effects (font (size 1.27 1.27)) hide)
     )
+    (property "variant" "Audio" (id 5) (at 161.29 60.96 0)
+      (effects (font (size 1.27 1.27)) hide)
+    )
     (pin "1")
     (pin "2")
@@
     )
     (property "LCSC" "" (id 4) (at 124.46 124.46 0)
+      (effects (font (size 1.27 1.27)) hide)
+    )
+    (property "DNP" "DNP" (id 5) (at 124.46 124.46 0)
+      (effects (font (size 1.27 1.27)) hide)
+    )
+    (property "variant" "Audio" (id 6) (at 124.46 124.46 0)
       (effects (font (size 1.27 1.27)) hide)
     )
@@
       (effects (font (size 1.27 1.27)) hide)
     )
+    (property "variant" "Audio" (id 5) (at 82.55 43.18 0)
+      (effects (font (size 1.27 1.27)) hide)
+    )
     (pin "1")
     (pin "2")
@@
       (effects (font (size 1.27 1.27)) hide)
     )
+    (property "DNP" "DNP" (id 5) (at 166.37 50.8 0)
+      (effects (font (size 1.27 1.27)) hide)
+    )
+    (property "variant" "Audio" (id 6) (at 166.37 50.8 0)
+      (effects (font (size 1.27 1.27)) hide)
+    )
     (pin "1")
     (pin "2")
@@
     )
     (property "LCSC" "C236994" (id 4) (at 255.27 115.57 0)
+      (effects (font (size 1.27 1.27)) hide)
+    )
+    (property "variant" "Audio" (id 5) (at 255.27 115.57 0)
       (effects (font (size 1.27 1.27)) hide)
     )
@@
       (effects (font (size 1.27 1.27)) hide)
     )
+    (property "variant" "Audio" (id 5) (at 113.03 43.18 0)
+      (effects (font (size 1.27 1.27)) hide)
+    )
     (pin "1")
     (pin "2")
@@
       (effects (font (size 1.27 1.27)) hide)
     )
+    (property "variant" "Audio" (id 5) (at 48.26 45.72 0)
+      (effects (font (size 1.27 1.27)) hide)
+    )
     (pin "1")
     (pin "2")
@@
     )
     (property "LCSC" "C389113" (id 4) (at 90.17 48.26 0)
+      (effects (font (size 1.27 1.27)) hide)
+    )
+    (property "variant" "Audio" (id 5) (at 90.17 48.26 0)
       (effects (font (size 1.27 1.27)) hide)
     )
@@
       (effects (font (size 1.27 1.27)) hide)
     )
+    (property "variant" "Audio" (id 5) (at 156.21 45.72 0)
+      (effects (font (size 1.27 1.27)) hide)
+    )
     (pin "1")
     (pin "2")
@@
       (effects (font (size 1.27 1.27)) hide)
     )
+    (property "DNP" "DNP" (id 5) (at 166.37 71.12 0)
+      (effects (font (size 1.27 1.27)) hide)
+    )
+    (property "variant" "Audio" (id 6) (at 166.37 71.12 0)
+      (effects (font (size 1.27 1.27)) hide)
+    )
     (pin "1")
     (pin "2")
@@
       (effects (font (size 1.27 1.27)) hide)
     )
+    (property "variant" "Audio" (id 5) (at 181.61 114.3 0)
+      (effects (font (size 1.27 1.27)) hide)
+    )
     (pin "1")
     (pin "2")
@@
     )
     (property "LCSC" "C105428" (id 4) (at 95.25 125.73 0)
+      (effects (font (size 1.27 1.27)) hide)
+    )
+    (property "variant" "Audio" (id 5) (at 95.25 125.73 0)
       (effects (font (size 1.27 1.27)) hide)
     )
@@
       (effects (font (size 1.27 1.27)) hide)
     )
+    (property "variant" "Audio" (id 5) (at 142.24 45.72 0)
+      (effects (font (size 1.27 1.27)) hide)
+    )
     (pin "5")
     (pin "6")
@@
       (effects (font (size 1.27 1.27)) hide)
     )
+    (property "DNP" "DNP" (id 5) (at 125.73 114.3 0)
+      (effects (font (size 1.27 1.27)) hide)
+    )
+    (property "variant" "Audio" (id 6) (at 125.73 114.3 0)
+      (effects (font (size 1.27 1.27)) hide)
+    )
     (pin "1")
     (pin "2")
@@
       (effects (font (size 1.27 1.27)) hide)
     )
+    (property "variant" "Audio" (id 5) (at 173.99 109.22 0)
+      (effects (font (size 1.27 1.27)) hide)
+    )
     (pin "1")
     (pin "2")
@@
     )
     (property "LCSC" "C389113" (id 4) (at 151.13 114.3 0)
+      (effects (font (size 1.27 1.27)) hide)
+    )
+    (property "variant" "Audio" (id 5) (at 151.13 114.3 0)
       (effects (font (size 1.27 1.27)) hide)
     )
@@
     )
     (property "LCSC" "C236994" (id 4) (at 203.2 111.76 0)
+      (effects (font (size 1.27 1.27)) hide)
+    )
+    (property "variant" "Audio" (id 5) (at 203.2 111.76 0)
       (effects (font (size 1.27 1.27)) hide)
     )
@@
       (effects (font (size 1.27 1.27)) hide)
     )
+    (property "variant" "Audio" (id 5) (at 177.8 66.04 0)
+      (effects (font (size 1.27 1.27)) hide)
+    )
     (pin "1")
     (pin "2")
@@
       (effects (font (size 1.27 1.27)) hide)
     )
+    (property "variant" "Audio" (id 5) (at 73.66 119.38 0)
+      (effects (font (size 1.27 1.27)) hide)
+    )
     (pin "1")
     (pin "2")
@@
       (effects (font (size 1.27 1.27)) hide)
     )
+    (property "variant" "Audio" (id 5) (at 73.66 106.68 0)
+      (effects (font (size 1.27 1.27)) hide)
+    )
     (pin "1")
     (pin "2")
@@
     )
     (property "LCSC" "C106246" (id 4) (at 120.65 48.26 0)
+      (effects (font (size 1.27 1.27)) hide)
+    )
+    (property "variant" "Audio" (id 5) (at 120.65 48.26 0)
       (effects (font (size 1.27 1.27)) hide)
     )
@@
       (effects (font (size 1.27 1.27)) hide)
     )
+    (property "variant" "Audio" (id 5) (at 213.36 59.69 0)
+      (effects (font (size 1.27 1.27)) hide)
+    )
     (pin "1")
     (pin "2")
@@
     )
     (property "LCSC" "C2922482" (id 4) (at 95.25 135.89 0)
+      (effects (font (size 1.27 1.27)) hide)
+    )
+    (property "variant" "Audio" (id 5) (at 95.25 135.89 0)
       (effects (font (size 1.27 1.27)) hide)
     )
@@
       (effects (font (size 1.27 1.27)) hide)
     )
+    (property "variant" "Audio" (id 5) (at 143.51 109.22 0)
+      (effects (font (size 1.27 1.27)) hide)
+    )
     (pin "1")
     (pin "2")
@@
       (effects (font (size 1.27 1.27)) hide)
     )
+    (property "variant" "Audio" (id 5) (at 241.3 115.57 0)
+      (effects (font (size 1.27 1.27)) hide)
+    )
     (pin "1")
     (pin "2")
@@
     )
     (property "LCSC" "C236994" (id 4) (at 227.33 59.69 0)
+      (effects (font (size 1.27 1.27)) hide)
+    )
+    (property "variant" "Audio" (id 5) (at 227.33 59.69 0)
       (effects (font (size 1.27 1.27)) hide)
     )
@@
       (effects (font (size 1.27 1.27)) hide)
     )
+    (property "variant" "Audio" (id 5) (at 114.3 109.22 0)
+      (effects (font (size 1.27 1.27)) hide)
+    )
     (pin "1")
     (pin "2")
@@
     )
     (property "LCSC" "C105428" (id 4) (at 135.89 134.62 0)
+      (effects (font (size 1.27 1.27)) hide)
+    )
+    (property "variant" "Audio" (id 5) (at 135.89 134.62 0)
       (effects (font (size 1.27 1.27)) hide)
     )
@@
       (effects (font (size 1.27 1.27)) hide)
     )
+    (property "variant" "Audio" (id 5) (at 97.79 43.18 0)
+      (effects (font (size 1.27 1.27)) hide)
+    )
     (pin "1")
     (pin "2")
@@
       (effects (font (size 1.27 1.27)) hide)
     )
+    (property "variant" "Audio" (id 5) (at 166.37 114.3 0)
+      (effects (font (size 1.27 1.27)) hide)
+    )
